File: audiokarma.brd (EAGLE design)
At the start: 100 x 80 mm, 70 parts, among them IC1 OPA2134U, IC2 OPA2134U

Commit message: rutado al 60%
Parts:
- removed IMP_L, IMP_R: 219-04, switch-dil:CTS-219-04
- removed LED1: (no value), led:LED5MM
- removed R31, R39: 3k3, rcl:R0805
- removed R32: 100, rcl:R0805
- removed R33: 16k, rcl:R0805
- removed R34: 2k2, rcl:R0805
- removed R35: 130, rcl:R0805
- removed R36, R38: 300, rcl:R0805
- removed R37: 180, rcl:R0805
- removed R40: 110k, rcl:R0805
- added JP1: (no value), pinhead:1X02
- added R13, R14: 3k3, rcl:R0805
- added R15: 16k, rcl:R0805
- added S1, S2: 219-04, switch-dil:CTS-219-04
- C1, C2: value 22UF -> 0-200p; device Panasonic-EEE0_EEE1_EEE2_EEEFC:CAPAE830X650N -> rcl:C0805
- C11, C12: value 68nF -> 100nF; device rcl:C050-035X075 -> rcl:C0805
- C13: value 47nF -> 100nF; device rcl:C050-025X075 -> rcl:C0805
- C14: value 1uF -> 100nF; device rcl:C050-050X075 -> rcl:C0805
- C15, C16: value 68nF -> 22UF; device rcl:C050-035X075 -> Panasonic-EEE0_EEE1_EEE2_EEEFC:CAPAE830X650N
- C17, C18: value 100nF -> 22UF; device rcl:C0805 -> Panasonic-EEE0_EEE1_EEE2_EEEFC:CAPAE830X650N
- C3, C4: value 22UF -> 47nF; device Panasonic-EEE0_EEE1_EEE2_EEEFC:CAPAE830X650N -> rcl:C050-025X075
- C5, C6: value 100nF -> 68nF; device rcl:C0805 -> rcl:C050-035X075
- C7, C8: value 47nF -> 68nF; device rcl:C050-025X075 -> rcl:C050-035X075
- R10: value 82k -> 100
- R11: value 33k -> 2k2
- R12: value (none) -> 100
- R16: value 3k3 -> 16k
- R17: value 100 -> 2k2
- R18: value 16k -> 130
- R2: value 2k2 -> 110k
- R22: value 180 -> 300
- R23: value 300 -> 180
- R24: value 3k3 -> 180
- R25: value 110k -> 300
- R26: value 150k -> 300
- R27: value 2k2 -> 3k3
- R28: value 110k -> 3k3
- R29: value 82k -> 110k
- R3: value (none) -> 150k
- R30: value 33k -> 110k
- R4: value (none) -> 110k
- R5, R7: value (none) -> 82k
- R6, R8: value (none) -> 33k
- R9: value 110k -> 2k2
- X1: device con-wago-500:W237-4 -> con-wago-500:W237-103
- moved X4 274.7 mm to (126.9, 62.8), flipped to the bottom, turned to 270 degrees
- moved R29 260.7 mm to (113.7, 75.5)
- moved R12 234.5 mm to (46.3, 47.8), turned to 90 degrees
- moved R30 233.2 mm to (112.6, 43.0), turned to 270 degrees
- moved C17 228.3 mm to (53.6, 67.2), turned to 90 degrees
- moved R26 218.1 mm to (81.7, 60.7)
- moved C13 208.2 mm to (63.1, 57.6), turned to 180 degrees
- moved R23 206.2 mm to (87.0, 92.8), turned to 270 degrees
- moved C18 204.6 mm to (52.5, 34.8), turned to 90 degrees
- moved C15 203.0 mm to (63.7, 67.2), turned to 90 degrees
- moved R21 201.4 mm to (90.0, 92.6), turned to 270 degrees
- moved R24 201.0 mm to (94.3, 50.0), turned to 90 degrees
- moved GAIN_R 200.3 mm to (92.2, 58.6)
- moved R28 196.8 mm to (55.6, 57.4), turned to 180 degrees
- moved R27 196.4 mm to (68.5, 56.9)
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Connections:
- removed net GND: C11.2, C12.2, C13.2, C15.2, C16.2, C7.2, R1.1, R10.1, R11.1, R17.1, R21.1, R22.1, R23.1, R25.1, R26.1, R28.1, R29.1, R30.1, R32.1, R36.1, R37.1, R38.1, R40.1, R9.1, X1.4, X2.2, X3.2
- removed net N$24: IMP_R.5, IMP_R.6, IMP_R.7, IMP_R.8, R27.1
- removed net N$33 (its old number): R34.1, R35.2
- removed net N$5: LED1.A, R12.2
- removed net N$6: IMP_L.5, IMP_L.6, IMP_L.7, IMP_L.8, R2.1, X1.1
- removed net V+: IC2.8
- new net INPUT_L: C1.1, R9.1, S1.5, S1.6, S1.7, S1.8, X1.1
- new net INPUT_R: C2.1, R11.1, S2.5, S2.6, S2.7, S2.8, X1.3
- new net N$23: R17.1, R18.2
- net AGND: now also C11.2, C12.1, C13.2, C14.1, C15.2, C16.1, C17.2, C2.2, C3.2, C7.2, C8.2, JP1.1, R1.1, R10.1, R12.1, R2.1, R21.1, R22.1, R23.1, R24.1, R25.1, R26.1, R29.1, R3.1, R30.1, R4.1, R5.1, R6.1, R7.1, R8.1, X1.2, X2.2, X3.2; no longer C17.1, C2.1, C3.1, LED1.K
- net N$1: now also S1.1; no longer IMP_L.1
- net N$12: now also IC2.7, R27.1; no longer IC2.1, R24.1
- net N$13: now also R3.2, S2.1; no longer IMP_R.1, R26.2
- net N$14: now also R9.2; no longer R2.2
- net N$15: now also R10.2, R13.1; no longer R16.1, R17.2
- net N$16: now also R29.2; no longer R25.2
- net N$17: now also R13.2, R15.2; no longer R16.2, R18.2
- net N$18: now also C3.1, IC2.5, R15.1, R17.2; no longer C7.1, IC2.3, R18.1, R19.2
- net N$19: now also R4.2, S2.2; no longer IMP_R.2, R28.2
- net N$2: now also R2.2, S1.2; no longer IMP_L.2, R9.2
- net N$20: now also R7.2, S2.3; no longer IMP_R.3, R29.2
- net N$21: now also R8.2, S2.4; no longer IMP_R.4, R30.2
- net N$22: now also C5.1, C7.1, R18.1; no longer C11.1, C12.1, R20.1
- net N$25: now also R11.2; no longer R27.2
- net N$26: now also IC2.6, R25.2, R27.2; no longer IC2.2, R23.2, R24.2
- net N$28: now also R23.2; no longer R22.2
- net N$29: now also R12.2, R14.1; no longer R31.1, R32.2
- net N$3: now also R5.2, S1.3; no longer IMP_L.3, R10.2
- net N$30: now also R14.2, R16.2; no longer R31.2, R33.2
- net N$31: now also C4.1, IC2.3, R16.1, R19.2; no longer C13.1, IC2.5, R33.1, R34.2
- net N$32: now also C6.1, C8.1, R20.1; no longer C15.1, C16.1, R35.1
- net N$34: now also IC2.2, R26.2, R28.2; no longer IC2.6, R38.2, R39.2
- net N$35: now also R22.2; no longer R36.2
- net N$36: now also R24.2; no longer R37.2
- net N$37: now also C10.1, IC2.1, R28.1; no longer C14.1, IC2.7, R39.1
- net N$38: now also C10.2, R30.2; no longer C14.2, R40.2
- net N$4: now also R6.2, S1.4; no longer IMP_L.4, R11.2
- net VCC: now also C11.1, C13.1, C15.1, C17.1, IC2.8; no longer C1.1, C4.1, C5.1, C6.1
- net VSS: now also C12.2, C14.2, C16.2, JP1.2; no longer C17.2, C2.2, C3.2, R12.1
Routing:
- added copper zone on layer 1, net AGND
- added copper zone on layer 16, net AGND
Other:
- board size 100 x 80 mm -> 162.2 x 102.9 mm

Commit message: colocados al 90%
Parts:
- moved H2 65.6 mm to (95.6, 55.8)
- moved H4 58.3 mm to (95.4, 6.77)
- moved R21 55.8 mm to (68.6, 41.1), turned to 90 degrees
- moved R23 54.2 mm to (72.5, 40.6), turned to 90 degrees
- moved X4 54.1 mm to (94.4, 19.5)
- moved C3 48.5 mm to (64.4, 23.0), turned to 180 degrees
- moved X2 47.3 mm to (96.3, 45.1)
- moved JP1 42.9 mm to (65.5, 15.4)
- moved R29 42.6 mm to (87.8, 41.7), turned to 90 degrees
- moved C9 40.2 mm to (81.8, 43.6), flipped to the bottom, turned to 180 degrees
- moved H1 38.4 mm to (6.03, 55.6)
- moved R24 35.3 mm to (60.2, 41.0)
- moved R22 34.7 mm to (57.8, 41.0)
- moved X3 34.6 mm to (96.2, 33.6)
- moved R1 34.5 mm to (15.0, 36.0), turned to 90 degrees
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Other:
- board size 162.2 x 102.9 mm -> 101.4 x 63.1 mm

Commit message: 95
Parts:
- moved X4 61.2 mm to (36.3, 38.6), turned to 0 degrees
- moved JP1 46.2 mm to (24.5, 36.9), flipped to the bottom, turned to 0 degrees
- moved X2 42.5 mm to (66.6, 14.7), turned to 270 degrees
- moved R29 37.7 mm to (58.7, 17.8), turned to 0 degrees
- moved H2 37.5 mm to (64.1, 35.4)
- moved C9 37.4 mm to (58.8, 14.0)
- moved H4 31.4 mm to (64.1, 4.62)
- moved X3 30.7 mm to (66.6, 25.1), turned to 270 degrees
- moved C13 30.0 mm to (48.4, 23.1)
- moved C5 28.7 mm to (54.6, 1.96)
- moved R30 27.8 mm to (61.9, 26.8)
- moved C10 27.7 mm to (58.0, 21.8)
- moved R18 24.3 mm to (49.9, 13.6), turned to 90 degrees
- moved C7 23.3 mm to (54.6, 6.06)
- moved R26 23.2 mm to (46.3, 27.1)
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Routing:
- removed copper zone on layer 1, net AGND
- removed copper zone on layer 16, net AGND
Other:
- board size 101.4 x 63.1 mm -> 72.3 x 42.2 mm

Commit message: rutado 100% pendiente revisión
Parts:
- moved C2 9.01 mm to (8.00, 10.0), turned to 270 degrees
- moved R12 3.00 mm to (32.5, 14.0)
- moved H2 2.96 mm to (67.0, 36.0)
- moved H4 2.93 mm to (67.0, 4.50)
- moved R14 2.50 mm to (32.5, 17.0), turned to 180 degrees
- moved R26 2.34 mm to (44.0, 27.0)
- moved R22 1.59 mm to (47.0, 27.0)
- moved H1 1.38 mm to (4.50, 36.0)
- moved R24 1.04 mm to (50.0, 27.0)
- moved X2 0.94 mm to (66.0, 14.0)
- moved R25 0.93 mm to (53.0, 27.0)
- moved R17 0.93 mm to (52.0, 13.5)
- moved R18 0.89 mm to (49.0, 13.5)
- moved C3 0.78 mm to (54.0, 9.85)
- moved C9 0.75 mm to (58.0, 14.0)
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Routing:
- net VSS: track 0.00 -> 72.2 mm, vias 0 -> 3
- net VCC: track 0.00 -> 55.6 mm, vias 0 -> 1
- net N$18: track 0.00 -> 44.3 mm, vias 0 -> 1
- net N$26: track 0.00 -> 38.6 mm, vias 0 -> 2
- net INPUT_L: track 0.00 -> 36.7 mm
- net N$34: track 0.00 -> 32.9 mm
- net INPUT_R: track 0.00 -> 29.5 mm
- net N$37: track 0.00 -> 23.1 mm, vias 0 -> 1
- net N$31: track 0.00 -> 17.6 mm
- net N$16: track 0.00 -> 12.6 mm
- net N$12: track 0.00 -> 12.3 mm
- net N$32: track 0.00 -> 11.8 mm
- net N$30: track 0.00 -> 11.6 mm
- net N$22: track 0.00 -> 11.6 mm
- net N$38: track 0.00 -> 10.6 mm
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- added copper zone on layer 1, net AGND
- added copper zone on layer 16, net AGND

Commit message: Phono100% e inicio de supply
Parts:
- renumbered GAIN_L to S3, GAIN_R to S4
Other:
- board size 72.3 x 42.2 mm -> 72 x 41 mm
- board text added: "AGND"
- board text added: "L"
- board text added: "R"
