File: audiokarma.sch (EAGLE design)
At the start: 70 parts, among them IC1 OPA2134U, IC2 OPA2134U

Commit message: rutado al 60%
Parts:
- removed LED1: (no value), led:LED5MM
- removed R32: 100, rcl:R-EU_R0805
- removed R33: 16k, rcl:R-EU_R0805
- removed R34: 2k2, rcl:R-EU_R0805
- removed R35: 130, rcl:R-EU_R0805
- removed R36, R38: 300, rcl:R-EU_R0805
- removed R37: 180, rcl:R-EU_R0805
- removed R39: 3k3, rcl:R-EU_R0805
- removed R40: 110k, rcl:R-EU_R0805
- added JP1: (no value), pinhead:PINHD-1X2
- added R13: 3k3, rcl:R-EU_R0805
- added R15: 16k, rcl:R-EU_R0805
- C1, C2: value 22UF -> 0-200p; device Panasonic-EEE0_EEE1_EEE2_EEEFC:EEE-FC1H220P-CASE-E -> rcl:C-EUC0805
- C11, C12: value 68nF -> 100nF; device rcl:C-EU050-035X075 -> rcl:C-EUC0805
- C13: value 47nF -> 100nF; device rcl:C-EU050-025X075 -> rcl:C-EUC0805
- C14: value 1uF -> 100nF; device rcl:C-EU050-050X075 -> rcl:C-EUC0805
- C15, C16: value 68nF -> 22UF; device rcl:C-EU050-035X075 -> Panasonic-EEE0_EEE1_EEE2_EEEFC:EEE-FC1H220P-CASE-E
- C17, C18: value 100nF -> 22UF; device rcl:C-EUC0805 -> Panasonic-EEE0_EEE1_EEE2_EEEFC:EEE-FC1H220P-CASE-E
- C3, C4: value 22UF -> 47nF; device Panasonic-EEE0_EEE1_EEE2_EEEFC:EEE-FC1H220P-CASE-E -> rcl:C-EU050-025X075
- C5, C6: value 100nF -> 68nF; device rcl:C-EUC0805 -> rcl:C-EU050-035X075
- C7, C8: value 47nF -> 68nF; device rcl:C-EU050-025X075 -> rcl:C-EU050-035X075
- R10: value 82k -> 100
- R11: value 33k -> 2k2
- R12: value (none) -> 100
- R16: value 3k3 -> 16k
- R17: value 100 -> 2k2
- R18: value 16k -> 130
- R2: value 2k2 -> 110k
- R22: value 180 -> 300
- R23: value 300 -> 180
- R24: value 3k3 -> 180
- R25: value 110k -> 300
- R26: value 150k -> 300
- R27: value 2k2 -> 3k3
- R28: value 110k -> 3k3
- R29: value 82k -> 110k
- R3: value (none) -> 150k
- R30: value 33k -> 110k
- R4: value (none) -> 110k
- R5, R7: value (none) -> 82k
- R6, R8: value (none) -> 33k
- R9: value 110k -> 2k2
- X1: device con-wago-500:W237-4 -> con-wago-500:W237-103
- renumbered IMP_L to S1, IMP_R to S2, R31 to R14
Connections:
- removed net GND: C11.2, C12.2, C13.2, C15.2, C16.2, C7.2, R1.1, R10.1, R11.1, R17.1, R21.1, R22.1, R23.1, R25.1, R26.1, R28.1, R29.1, R30.1, R32.1, R36.1, R37.1, R38.1, R40.1, R9.1, X1-4.KL, X2-2.KL, X3-2.KL
- removed net N$24: R27.1, S2.5, S2.6, S2.7, S2.8
- removed net N$33 (its old number): R34.1, R35.2
- removed net N$5: LED1.A, R12.2
- removed net N$6: R2.1, S1.5, S1.6, S1.7, S1.8, X1-1.KL
- new net INPUT_L: C1.1, R9.1, S1.5, S1.6, S1.7, S1.8, X1-1.KL
- new net INPUT_R: C2.1, R11.1, S2.5, S2.6, S2.7, S2.8, X1-3.KL
- new net N$23: R17.1, R18.2
- net AGND: now also C11.2, C12.1, C13.2, C14.1, C15.2, C16.1, C17.2, C2.2, C3.2, C7.2, C8.2, JP1.1, R1.1, R10.1, R12.1, R2.1, R21.1, R22.1, R23.1, R24.1, R25.1, R26.1, R29.1, R3.1, R30.1, R4.1, R5.1, R6.1, R7.1, R8.1, X1-2.KL, X2-2.KL, X3-2.KL; no longer C17.1, C2.1, C3.1, LED1.C
- net N$12: now also IC2B.OUT, R27.1; no longer IC2A.OUT, R24.1
- net N$13: now also R3.2; no longer R26.2
- net N$14: now also R9.2; no longer R2.2
- net N$15: now also R10.2, R13.1; no longer R16.1, R17.2
- net N$16: now also R29.2; no longer R25.2
- net N$17: now also R13.2, R15.2; no longer R16.2, R18.2
- net N$18: now also C3.1, IC2B.+IN, R15.1, R17.2; no longer C7.1, IC2A.+IN, R18.1, R19.2
- net N$19: now also R4.2; no longer R28.2
- net N$2: now also R2.2; no longer R9.2
- net N$20: now also R7.2; no longer R29.2
- net N$21: now also R8.2; no longer R30.2
- net N$22: now also C5.1, C7.1, R18.1; no longer C11.1, C12.1, R20.1
- net N$25: now also R11.2; no longer R27.2
- net N$26: now also IC2B.-IN, R25.2, R27.2; no longer IC2A.-IN, R23.2, R24.2
- net N$28: now also R23.2; no longer R22.2
- net N$29: now also R12.2; no longer R32.2
- net N$3: now also R5.2; no longer R10.2
- net N$30: now also R16.2; no longer R33.2
- net N$31: now also C4.1, IC2A.+IN, R16.1, R19.2; no longer C13.1, IC2B.+IN, R33.1, R34.2
- net N$32: now also C6.1, C8.1, R20.1; no longer C15.1, C16.1, R35.1
- net N$34: now also IC2A.-IN, R26.2, R28.2; no longer IC2B.-IN, R38.2, R39.2
- net N$35: now also R22.2; no longer R36.2
- net N$36: now also R24.2; no longer R37.2
- net N$37: now also C10.1, IC2A.OUT, R28.1; no longer C14.1, IC2B.OUT, R39.1
- net N$38: now also C10.2, R30.2; no longer C14.2, R40.2
- net N$4: now also R6.2; no longer R11.2
- net VCC: now also C11.1, C13.1, C15.1, C17.1, IC2A.V+; no longer C1.1, C4.1, C5.1, C6.1
- net VSS: now also C12.2, C14.2, C16.2, JP1.2; no longer C17.2, C2.2, C3.2, R12.1
Other:
- moved on the sheet: C10, C11, C12, C13, C14, C5, C6, C7, C8, IC2A, IC2B, R12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

Commit message: Phono100% e inicio de supply
Parts:
- renumbered GAIN_L to S3, GAIN_R to S4
Other:
- moved on the sheet: H1, H2, H3, H4
Changed lines of the file:
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@@
 <part name="R23" library="rcl" deviceset="R-EU_" device="R0805" value="180"/>
 <part name="R25" library="rcl" deviceset="R-EU_" device="R0805" value="300"/>
-<part name="GAIN_L" library="switch-dil" deviceset="219-02*" device=""/>
+<part name="S3" library="switch-dil" deviceset="219-02*" device=""/>
 <part name="R27" library="rcl" deviceset="R-EU_" device="R0805" value="3k3"/>
 <part name="R29" library="rcl" deviceset="R-EU_" device="R0805" value="110k"/>
@@
 <part name="R24" library="rcl" deviceset="R-EU_" device="R0805" value="180"/>
 <part name="R26" library="rcl" deviceset="R-EU_" device="R0805" value="300"/>
-<part name="GAIN_R" library="switch-dil" deviceset="219-02*" device=""/>
+<part name="S4" library="switch-dil" deviceset="219-02*" device=""/>
 <part name="R28" library="rcl" deviceset="R-EU_" device="R0805" value="3k3"/>
 <part name="R30" library="rcl" deviceset="R-EU_" device="R0805" value="110k"/>
@@
 <part name="C1" library="rcl" deviceset="C-EU" device="C0805" value="0-200p"/>
 <part name="C2" library="rcl" deviceset="C-EU" device="C0805" value="0-200p"/>
-<part name="SUPPLY10" library="supply2" deviceset="AGND" device=""/>
-<part name="SUPPLY11" library="supply2" deviceset="AGND" device=""/>
+<part name="SUPPLY1" library="supply2" deviceset="AGND" device=""/>
+<part name="SUPPLY2" library="supply2" deviceset="AGND" device=""/>
 <part name="JP1" library="pinhead" deviceset="PINHD-1X2" device=""/>
 </parts>
@@
 <attribute name="VALUE" x="181.102" y="54.61" size="1.778" layer="96" rot="R90"/>
 </instance>
-<instance part="H1" gate="G$1" x="45.72" y="114.3"/>
+<instance part="H1" gate="G$1" x="213.36" y="132.08"/>
 <instance part="R13" gate="G$1" x="233.68" y="71.12"/>
 <instance part="R10" gate="G$1" x="215.9" y="60.96" rot="R90"/>
@@
 <instance part="R23" gate="G$1" x="309.88" y="53.34" rot="R90"/>
 <instance part="R25" gate="G$1" x="320.04" y="58.42" rot="R90"/>
-<instance part="GAIN_L" gate="G$1" x="304.8" y="71.12"/>
+<instance part="S3" gate="G$1" x="304.8" y="71.12"/>
 <instance part="R27" gate="G$1" x="332.74" y="78.74" rot="R180"/>
 <instance part="R29" gate="G$1" x="363.22" y="68.58" rot="R90"/>
@@
 <instance part="R24" gate="G$1" x="314.96" y="-22.86" rot="R90"/>
 <instance part="R26" gate="G$1" x="325.12" y="-22.86" rot="R90"/>
-<instance part="GAIN_R" gate="G$1" x="309.88" y="-5.08"/>
+<instance part="S4" gate="G$1" x="309.88" y="-5.08"/>
 <instance part="R28" gate="G$1" x="337.82" y="2.54" rot="R180"/>
 <instance part="R30" gate="G$1" x="368.3" y="-12.7" rot="R90"/>
@@
 <instance part="SUPPLY5" gate="G$1" x="297.18" y="33.02"/>
 <instance part="SUPPLY6" gate="G$1" x="299.72" y="10.16"/>
-<instance part="H2" gate="G$1" x="81.28" y="119.38"/>
-<instance part="H3" gate="G$1" x="116.84" y="121.92"/>
-<instance part="H4" gate="G$1" x="157.48" y="124.46"/>
+<instance part="H2" gate="G$1" x="213.36" y="124.46"/>
+<instance part="H3" gate="G$1" x="238.76" y="132.08"/>
+<instance part="H4" gate="G$1" x="238.76" y="124.46"/>
 <instance part="X1" gate="-1" x="106.68" y="91.44" smashed="yes">
 <attribute name="NAME" x="106.68" y="92.329" size="1.778" layer="95" rot="R180"/>
@@
 <instance part="C1" gate="G$1" x="129.54" y="71.12"/>
 <instance part="C2" gate="G$1" x="144.78" y="-12.7"/>
-<instance part="SUPPLY10" gate="G$1" x="167.64" y="35.56"/>
-<instance part="SUPPLY11" gate="G$1" x="172.72" y="-45.72"/>
+<instance part="SUPPLY1" gate="G$1" x="167.64" y="35.56"/>
+<instance part="SUPPLY2" gate="G$1" x="172.72" y="-45.72"/>
 <instance part="JP1" gate="G$1" x="563.88" y="30.48"/>
 </instances>
@@
 <segment>
 <wire x1="284.48" y1="93.98" x2="284.48" y2="78.74" width="0.1524" layer="91"/>
-<pinref part="GAIN_L" gate="G$1" pin="4"/>
+<pinref part="S3" gate="G$1" pin="4"/>
 <wire x1="284.48" y1="78.74" x2="304.8" y2="78.74" width="0.1524" layer="91"/>
-<pinref part="GAIN_L" gate="G$1" pin="3"/>
+<pinref part="S3" gate="G$1" pin="3"/>
 <wire x1="304.8" y1="78.74" x2="307.34" y2="78.74" width="0.1524" layer="91"/>
 <wire x1="307.34" y1="78.74" x2="320.04" y2="78.74" width="0.1524" layer="91"/>
@@
 <net name="N$27" class="0">
 <segment>
-<pinref part="GAIN_L" gate="G$1" pin="1"/>
+<pinref part="S3" gate="G$1" pin="1"/>
 <pinref part="R21" gate="G$1" pin="2"/>
 <wire x1="304.8" y1="63.5" x2="302.26" y2="63.5" width="0.1524" layer="91"/>
@@
 <net name="N$28" class="0">
 <segment>
-<pinref part="GAIN_L" gate="G$1" pin="2"/>
+<pinref part="S3" gate="G$1" pin="2"/>
 <pinref part="R23" gate="G$1" pin="2"/>
 <wire x1="307.34" y1="63.5" x2="309.88" y2="63.5" width="0.1524" layer="91"/>
@@
 <segment>
 <wire x1="289.56" y1="17.78" x2="289.56" y2="2.54" width="0.1524" layer="91"/>
-<pinref part="GAIN_R" gate="G$1" pin="4"/>
+<pinref part="S4" gate="G$1" pin="4"/>
 <wire x1="289.56" y1="2.54" x2="309.88" y2="2.54" width="0.1524" layer="91"/>
-<pinref part="GAIN_R" gate="G$1" pin="3"/>
+<pinref part="S4" gate="G$1" pin="3"/>
 <wire x1="309.88" y1="2.54" x2="312.42" y2="2.54" width="0.1524" layer="91"/>
 <wire x1="312.42" y1="2.54" x2="325.12" y2="2.54" width="0.1524" layer="91"/>
@@
 <net name="N$35" class="0">
 <segment>
-<pinref part="GAIN_R" gate="G$1" pin="1"/>
+<pinref part="S4" gate="G$1" pin="1"/>
 <pinref part="R22" gate="G$1" pin="2"/>
 <wire x1="309.88" y1="-12.7" x2="307.34" y2="-12.7" width="0.1524" layer="91"/>
@@
 <net name="N$36" class="0">
 <segment>
-<pinref part="GAIN_R" gate="G$1" pin="2"/>
+<pinref part="S4" gate="G$1" pin="2"/>
 <pinref part="R24" gate="G$1" pin="2"/>
 <wire x1="312.42" y1="-12.7" x2="314.96" y2="-12.7" width="0.1524" layer="91"/>
@@
 <wire x1="160.02" y1="45.72" x2="129.54" y2="45.72" width="0.1524" layer="91"/>
 <wire x1="129.54" y1="45.72" x2="129.54" y2="66.04" width="0.1524" layer="91"/>
-<pinref part="SUPPLY10" gate="G$1" pin="AGND"/>
+<pinref part="SUPPLY1" gate="G$1" pin="AGND"/>
 </segment>
 <segment>
@@
 <pinref part="C2" gate="G$1" pin="2"/>
 <wire x1="144.78" y1="-35.56" x2="144.78" y2="-17.78" width="0.1524" layer="91"/>
-<pinref part="SUPPLY11" gate="G$1" pin="AGND"/>
-</segment>
-</net>
+<pinref part="SUPPLY2" gate="G$1" pin="AGND"/>
+</segment>
+</net>
